File: pcb/MGC_module.kicad_sch (KiCad schematic)
At the start: 48 parts, among them J1 Micro_SD_Card, J11 103P012BB100, J12 103P012BB100, J13 103P012BB100, J3 103P012BB100, J7 103P012BB100, SW1 SW_DIP_x02, U1 ESP32-WROOM-32UE-R2, U2 74AHC1G02, U5 MCP23018x-x-SS

Commit message: Add missing vendor(id)
Parts:
- J1: DigiKey (none) -> WM6698CT-ND
- R10, R11, R13, R6, R9: HTL (none) -> 102967
- R12: HTL (none) -> 102961
- R14: HTL (none) -> 102962
- R15: HTL (none) -> 102960
- R18, R19: HTL 102934 -> 102902
- R3: HTL 102934 -> 102959
- R7: HTL (none) -> 102987
- U1: DigiKey (none) -> 1965-ESP32-WROOM-32UE-N4CT-ND, WM12219-ND
- U2: DigiKey (none) -> 296-8742-1-ND
- U5: DigiKey (none) -> 150-MCP23018T-E/SSCT-ND
Changed lines of the file:
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@@
 			)
 		)
+		(property "DigiKey" "150-MCP23018T-E/SSCT-ND"
+			(at 120.65 175.26 0)
+			(effects
+				(font
+					(size 1.27 1.27)
+				)
+				(hide yes)
+			)
+		)
 		(pin "11"
 		)
@@
 			)
 		)
+		(property "HTL" "102967"
+			(at 144.78 100.33 90)
+			(effects
+				(font
+					(size 1.27 1.27)
+				)
+				(hide yes)
+			)
+		)
 		(pin "2"
 		)
@@
 			)
 		)
+		(property "HTL" "102960"
+			(at 152.4 160.02 90)
+			(effects
+				(font
+					(size 1.27 1.27)
+				)
+				(hide yes)
+			)
+		)
 		(pin "2"
 		)
@@
 			)
 		)
+		(property "HTL" "102967"
+			(at 137.16 100.33 90)
+			(effects
+				(font
+					(size 1.27 1.27)
+				)
+				(hide yes)
+			)
+		)
 		(pin "2"
 		)
@@
 			)
 		)
-		(property "HTL" "102934"
+		(property "HTL" "102902"
 			(at 102.87 129.54 90)
 			(effects
@@
 			)
 		)
+		(property "HTL" "102967"
+			(at 139.7 100.33 90)
+			(effects
+				(font
+					(size 1.27 1.27)
+				)
+				(hide yes)
+			)
+		)
 		(pin "2"
 		)
@@
 			)
 		)
+		(property "HTL" "102967"
+			(at 40.64 93.98 90)
+			(effects
+				(font
+					(size 1.27 1.27)
+				)
+				(hide yes)
+			)
+		)
 		(pin "2"
 		)
@@
 			)
 		)
-		(property "HTL" "102934"
+		(property "HTL" "102959"
 			(at 214.63 90.17 90)
 			(effects
@@
 			)
 		)
+		(property "DigiKey" "WM6698CT-ND"
+			(at 200.66 114.3 0)
+			(effects
+				(font
+					(size 1.27 1.27)
+				)
+				(hide yes)
+			)
+		)
 		(pin "7"
 		)
@@
 			)
 		)
+		(property "HTL" "102987"
+			(at 44.45 93.98 90)
+			(effects
+				(font
+					(size 1.27 1.27)
+				)
+				(hide yes)
+			)
+		)
 		(pin "2"
 		)
@@
 			)
 		)
-		(property "HTL" "102934"
+		(property "HTL" "102902"
 			(at 102.87 132.08 90)
 			(effects
@@
 			)
 		)
+		(property "DigiKey" "296-8742-1-ND"
+			(at 124.46 142.24 0)
+			(effects
+				(font
+					(size 1.27 1.27)
+				)
+				(hide yes)
+			)
+		)
 		(pin "5"
 		)
@@
 			)
 		)
+		(property "HTL" "102967"
+			(at 134.62 100.33 90)
+			(effects
+				(font
+					(size 1.27 1.27)
+				)
+				(hide yes)
+			)
+		)
 		(pin "2"
 		)
@@
 			)
 		)
+		(property "HTL" "102961"
+			(at 142.24 100.33 90)
+			(effects
+				(font
+					(size 1.27 1.27)
+				)
+				(hide yes)
+			)
+		)
 		(pin "2"
 		)
@@
 			)
 		)
+		(property "HTL" "102962"
+			(at 152.4 149.86 90)
+			(effects
+				(font
+					(size 1.27 1.27)
+				)
+				(hide yes)
+			)
+		)
 		(pin "2"
 		)
@@
 			(at 74.93 124.46 0)
 			(effects
+				(font
+					(size 1.27 1.27)
+				)
+				(hide yes)
+			)
+		)
+		(property "DigiKey" "1965-ESP32-WROOM-32UE-N4CT-ND, WM12219-ND"
+			(at 74.93 124.46 0)
+			(effects
